Commit message: Custom humble setup for my robot

File: linorobot2_description/urdf/2wd_properties.urdf.xacro (robot description, xacro)
@@ -1,20 +1,21 @@
 <?xml version="1.0"?>
 <robot xmlns:xacro="http://ros.org/wiki/xacro">
-  <xacro:property name="base_length" value="0.24" />
-  <xacro:property name="base_width" value="0.275" />
-  <xacro:property name="base_height" value="0.003" />
-  <xacro:property name="base_mass" value="1" />
-  <xacro:property name="wheel_radius" value="0.045" />
-  <xacro:property name="wheel_width" value="0.01" />
+  <xacro:property name="base_length" value="0.1435" />
+  <xacro:property name="base_width" value="0.1435" />
+  <xacro:property name="base_height" value="0.156" />
+  <xacro:property name="base_mass" value="1.2" />
+  <xacro:property name="wheel_radius" value="0.033" />
+  <xacro:property name="wheel_width" value="0.027" />
   <xacro:property name="wheel_pos_x" value="0.0" />
-  <xacro:property name="wheel_pos_y" value="0.13" />
-  <xacro:property name="wheel_pos_z" value="-0.03" />
-  <xacro:property name="wheel_mass" value=".1" />
-  <xacro:property name="wheel_torque" value="20" />
-  <xacro:property name="front_caster_wheel" value="true" />
+  <xacro:property name="wheel_pos_y" value="0.08675" />
+  <xacro:property name="wheel_pos_z" value="0.0238" />
+  <xacro:property name="wheel_mass" value="0.0334" />
+  <xacro:property name="wheel_torque" value="0.43" />
+  <xacro:property name="front_caster_wheel" value="false" />
   <xacro:property name="rear_caster_wheel" value="true" />
   <xacro:property name="laser_pose">
-    <origin xyz="0.12 0 0.33" rpy="0 0 0"/>
+    <origin xyz="-0.0331 0 0.208" rpy="0 0 0"/>
   </xacro:property>
+  <!-- Unused -->
   <xacro:property name="depth_sensor_pose">
     <origin xyz="0.14 0.0 0.045" rpy="0 0 0"/>
@@ -23,3 +24,4 @@
     <origin xyz="-0.14 0.0 0.045" rpy="0 0 3.14159"/>
   </xacro:property>
+  <!-- Unused -->
 </robot>

File: linorobot2_description/urdf/mech/base.urdf.xacro (robot description, xacro)
@@ -5,15 +5,16 @@
     <link name="base_link">
       <visual>
-        <origin xyz="0 0 0" rpy="0 0 0"/>
+        <origin xyz="-0.0276 0 0" rpy="0 0 0"/>
         <geometry>
-          <box size="${length} ${width} ${height}"/>
+          <!-- <box size="${length} ${width} ${height}"/> -->
           <!-- <mesh filename="" scale="0.001 0.001 0.001"/> -->
+          <mesh filename="package://linorobot2_description/meshes/lino_base.STL" scale="0.001 0.001 0.001"/>
         </geometry>
-        <material name="yellow">
-          <color rgba="0.8784 0.6627 0.6627 1.0"/>
+        <material name="light_black">
+          <color rgba="0.4 0.4 0.4 1.0"/>
         </material>
       </visual>
       <collision>
-        <origin xyz="0 0 0" rpy="0 0 0"/>
+        <origin xyz="-0.0276 0 ${height/2}" rpy="0 0 0"/>
         <geometry>
           <box size="${length} ${width} ${height}"/>
@@ -21,9 +22,9 @@
       </collision>
       <inertial>
-        <origin xyz="0 0 0" rpy="0 0 0"/>
+        <origin xyz="-0.02957230 -0.00249250 0.04657955" rpy="0 0 0"/>
         <mass value="${mass}"/>
-        <inertia ixx="${(1/12) * mass * ((width  * width)  + (height * height))}" ixy="0.0" ixz="0.0"
-                 iyy="${(1/12) * mass * ((length * length) + (height * height))}" iyz="0.0"
-                 izz="${(1/12) * mass * ((length * length) + (width  * width))}"/>
+        <inertia ixx="0.00382227" ixy="-0.00007090" ixz="-0.00008756"
+                 iyy="0.00381152" iyz="-0.00003095"
+                 izz="0.00291391"/>
       </inertial>
     </link>
@@ -31,15 +32,21 @@
       <visual>
         <material>
-          <ambient>0.8392 0.6314 0.0 1.0</ambient>
+          <!-- <ambient>0.8392 0.6314 0.0 1.0</ambient>
           <diffuse>0.8392 0.6314 0.0 1.0</diffuse>
           <specular>0.99 0.99 0.99 1.0</specular>
           <emissive>0.0 0.0 0.0 0.0</emissive>
+          <ambient>0.4 0.4 0.4 1.0</ambient>   -->
+          <!-- <ambient>0.4 0.4 0.4 1.0</ambient>
+          <diffuse>0.4 0.4 0.4 1.0</diffuse>
+          <specular>0.2 0.2 0.2 1.0</specular>
+          <emissive>0.0 0.0 0.0 0.0</emissive> -->
         </material>
       </visual>
+      <material>Gazebo/White</material>
     </gazebo>
     <joint name="base_to_footprint" type="fixed">
       <parent link="base_footprint"/>
       <child link="base_link"/>
-      <origin xyz="0 0 ${wheel_radius - wheel_pos_z}" rpy="0 0 0"/>
+      <origin xyz="0 0 0.0092" rpy="0 0 0"/>
     </joint>
   </xacro:macro>

File: linorobot2_description/urdf/mech/caster_wheel.urdf.xacro (robot description, xacro)
@@ -2,10 +2,10 @@
 <robot xmlns:xacro="http://ros.org/wiki/xacro">
   <xacro:macro name="caster_wheel" params="side mass base_length wheel_radius wheel_pos_z">
-    <xacro:property name="caster_wheel_radius" value="${(wheel_radius - wheel_pos_z) / 2}" />
+    <xacro:property name="caster_wheel_radius" value="0.0075" />
     <xacro:if value="${side == 'front'}">
         <xacro:property name="caster_wheel_x" value="${(base_length / 2) - caster_wheel_radius}" />
     </xacro:if>
     <xacro:if value="${side == 'rear'}">
-        <xacro:property name="caster_wheel_x" value="${-(base_length / 2) + caster_wheel_radius}" />
+        <xacro:property name="caster_wheel_x" value="-0.0661" />
     </xacro:if>
     <link name="${side}_caster_wheel_link">
@@ -15,6 +15,6 @@
           <sphere radius="${caster_wheel_radius}" />
         </geometry>
-        <material name="black">
-            <color rgba="0.0 0.0 0.0 1.0"/>
+        <material name="white">
+          <color rgba="1.0 1.0 1.0 1.0"/>
         </material>
       </visual>
@@ -40,5 +40,5 @@
       <parent link="base_link"/>
       <child link="${side}_caster_wheel_link"/>
-      <origin xyz="${caster_wheel_x} 0 -${caster_wheel_radius}" rpy="0 0 0"/>
+      <origin xyz="${caster_wheel_x} 0 -0.002" rpy="0 0 0"/>
     </joint>
   </xacro:macro>

File: linorobot2_description/urdf/mech/wheel.urdf.xacro (robot description, xacro)
@@ -4,10 +4,11 @@
     <link name="${side}_wheel_link">
       <visual>
-        <origin xyz="0 0 0" rpy="${pi/2} 0 0"/>
+        <origin xyz="0 0 0" rpy="0 0 0"/>
         <geometry>
-          <cylinder radius="${radius}" length="${width}"/>
+          <!-- <cylinder radius="${radius}" length="${width}"/> -->
+          <mesh filename="package://linorobot2_description/meshes/wheel_${side}.STL" scale="0.001 0.001 0.001"/>
         </geometry>
-        <material name="blue">
-            <color rgba="0.1764 0.4588 0.8509 1.0"/>
+        <material name="dark">
+          <color rgba="0.3 0.3 0.3 1.0"/>
         </material>
       </visual>
@@ -21,7 +22,7 @@
         <origin xyz="0 0 0" rpy="0 0 0"/>
         <mass value="${mass}"/>
-        <inertia ixx="${(2/5) * mass * (radius * radius)}" ixy="0" ixz="0"
-                 iyy="${(2/5) * mass * (radius * radius)}" iyz="0"
-                 izz="${(2/5) * mass * (radius * radius)}" />
+        <inertia ixx="${(1/12) * mass * (3*radius*radius + width*width)}" ixy="0" ixz="0"
+                 iyy="${(1/2) * mass * (radius*radius)}" iyz="0"
+                 izz="${(1/12) * mass * (3*radius*radius + width*width)}" />
       </inertial>
     </link>
@@ -29,10 +30,15 @@
       <visual>
         <material>
-          <ambient>0.1764 0.4588 0.8509 1.0</ambient>
+          <!-- <ambient>0.1764 0.4588 0.8509 1.0</ambient>
           <diffuse>0.1764 0.4588 0.8509 1.0</diffuse>
           <specular>0.1764 0.4588 0.8509 1.0</specular>
-          <emissive>0.0 0.0 0.0 0.0</emissive>
+          <emissive>0.0 0.0 0.0 0.0</emissive>   -->
+          <!-- <ambient>0.3 0.3 0.3 1.0</ambient>
+          <diffuse>0.3 0.3 0.3 1.0</diffuse>
+          <specular>0.05 0.05 0.05 1.0</specular>
+          <emissive>0.0 0.0 0.0 0.0</emissive> -->
         </material>
       </visual>
+      <material>Gazebo/FlatBlack</material>
     </gazebo>
     <joint name="${side}_wheel_joint" type="continuous">

File: linorobot2_description/urdf/robots/2wd.urdf.xacro (robot description, xacro)
@@ -7,6 +7,6 @@
   <xacro:include filename="$(find linorobot2_description)/urdf/sensors/imu.urdf.xacro" />
   <xacro:include filename="$(find linorobot2_description)/urdf/sensors/generic_laser.urdf.xacro" />
-  <xacro:include filename="$(find linorobot2_description)/urdf/sensors/depth_sensor.urdf.xacro" />
-  <xacro:include filename="$(find linorobot2_description)/urdf/sensors/camera.urdf.xacro" />
+  <!-- <xacro:include filename="$(find linorobot2_description)/urdf/sensors/depth_sensor.urdf.xacro" /> -->
+  <!-- <xacro:include filename="$(find linorobot2_description)/urdf/sensors/camera.urdf.xacro" /> -->
   <xacro:include filename="$(find linorobot2_description)/urdf/controllers/diff_drive.urdf.xacro" />
   <xacro:base
@@ -58,13 +58,13 @@
     <xacro:insert_block name="laser_pose" />
   </xacro:generic_laser>
-  <xacro:depth_sensor>
+  <!-- <xacro:depth_sensor>
     <xacro:insert_block name="depth_sensor_pose" />
-  </xacro:depth_sensor>
-  <xacro:rgb_camera
+  </xacro:depth_sensor> -->
+  <!-- <xacro:rgb_camera
       parent="base_link"
       name="rear_rgb_camera"
       topic_name="rear_rgb_camera/image">
     <xacro:insert_block name="rear_camera_sensor_pose" />
-  </xacro:rgb_camera>
+  </xacro:rgb_camera> -->
   <xacro:diff_drive_controller
     wheel_separation="${wheel_pos_y * 2}"

File: linorobot2_description/urdf/sensors/imu.urdf.xacro (robot description, xacro)
@@ -5,5 +5,5 @@
       <parent link="base_link"/>
       <child link="imu_link"/>
-      <origin xyz="0 0 0" rpy="0 0 0"/>
+      <origin xyz="-0.07682 0 0.0826" rpy="0 0 0"/>
     </joint>
     <gazebo reference="imu_link">

File: linorobot2_description/urdf/sensors/laser.urdf.xacro (robot description, xacro)
@@ -1,27 +1,31 @@
 <robot xmlns:xacro="http://ros.org/wiki/xacro">
   <xacro:property name="M_PI" value="3.1415926535897931" />
+  <xacro:property name="ld_radius" value="0.04" />
+  <xacro:property name="ld_height" value="0.05" />
+  <xacro:property name="ld_mass" value="0.16" />
   <xacro:macro name="laser" params="*origin update_rate ray_count min_angle max_angle min_range max_range frame_id topic_name">
     <link name="${frame_id}">
       <visual>
-        <origin xyz="0 0 -0.025" rpy="0 0 0"/>
+        <origin xyz="0 0 0" rpy="0 0 0"/>
         <geometry>
-          <cylinder radius="0.0375" length="0.05"/>
+          <!-- <cylinder radius="0.0375" length="0.05"/> -->
+          <mesh filename="package://linorobot2_description/meshes/lds.stl" scale="0.001 0.001 0.001"/>
         </geometry>
-        <material name="green">
-            <color rgba="0.003 0.639 0.223 1.0"/>
+        <material name="dark">
+          <color rgba="0.3 0.3 0.3 1.0"/>
         </material>
       </visual>
       <collision>
-        <origin xyz="0 0 -0.025" rpy="0 0 0"/>
+        <origin xyz="0.015 0 -0.015" rpy="0 0 0"/>
         <geometry>
-          <cylinder radius="0.0375" length="0.05"/>
+          <cylinder radius="${ld_radius}" length="${ld_height}"/>
         </geometry>
       </collision>
       <inertial>
         <origin xyz="0 0 0" rpy="0 0 0"/>
-        <mass value="0.1"/>
-        <inertia ixx="${(2/5) * 0.1 * (0.0375 * 0.0375)}" ixy="0" ixz="0"
-                 iyy="${(2/5) * 0.1 * (0.0375 * 0.0375)}" iyz="0"
-                 izz="${(2/5) * 0.1 * (0.0375 * 0.0375)}" />
+        <mass value="${ld_mass}"/>
+        <inertia ixx="${(1/12) * ld_mass * (3*ld_radius*ld_radius + ld_height*ld_height)}" ixy="0" ixz="0"
+                 iyy="${(1/12) * ld_mass * (3*ld_radius*ld_radius + ld_height*ld_height)}" iyz="0"
+                 izz="${(1/2) * ld_mass * (ld_radius*ld_radius)}" />
       </inertial>
     </link>
@@ -29,10 +33,15 @@
       <visual>
         <material>
-          <ambient>0.003 0.639 0.223 1.0</ambient>
+          <!-- <ambient>0.003 0.639 0.223 1.0</ambient>
           <diffuse>0.003 0.639 0.223 1.0</diffuse>
           <specular>0.003 0.639 0.223 1.0</specular>
-          <emissive>0.0 0.0 0.0 0.0</emissive>
+          <emissive>0.0 0.0 0.0 0.0</emissive>   -->
+          <!-- <ambient>0.3 0.3 0.3 1.0</ambient>
+          <diffuse>0.3 0.3 0.3 1.0</diffuse>
+          <specular>0.1 0.1 0.1 1.0</specular>
+          <emissive>0.0 0.0 0.0 0.0</emissive> -->
         </material>
       </visual>
+      <material>Gazebo/FlatBlack</material>
     </gazebo>
     <joint name="${frame_id}_to_base_link" type="fixed">
